File: dsi-shield-bga/power.sch (KiCad schematic (older format))
At the start: 25 parts, among them IC1 LM26480

Commit message: datasheet
Parts:
- added C16: 10u, Capacitor_SMD:C_0603_1608Metric, symbol dsi_shield:Cap
- added C17: 100n, Capacitor_SMD:C_0402_1005Metric, symbol dsi_shield:Cap
- added P1: USB_C_Plug, Connector_USB:USB_C_Receptacle_Amphenol_12401548E4-2A, symbol Connector:USB_C_Plug
- added U4: CH340E, Package_SO:MSOP-10-1EP_3x3mm_P0.5mm_EP1.68x1.88mm_ThermalVias, symbol mybays:CH340E
Connections:
- net +5V: now also C16.1, P1.A4 (VBUS), P1.A9 (VBUS), P1.B4 (VBUS), P1.B9 (VBUS), U4.7 (VCC)
- net GND: now also C16.2, C17.1, U4.3 (GND)
- new net: P1.A6 (D+), U4.1 (UD+)
- new net: C17.2, U4.10 (V3)
- new net: P1.A7 (D-), U4.2 (UD-)
- new net: P1.A1 (GND), P1.A12 (GND), P1.B1 (GND), P1.B12 (GND)
- new net RXD: U4.9 (RXD)
- new net TXD: U4.8 (TXD)
Changed lines of the file:
@@
 U 1 1 5F14C81C
 P 3350 1400
-F 0 "R11" H 3450 1501 50  0000 C CNN
-F 1 "100k" H 3450 1402 60  0000 C CNN
+F 0 "R11" H 3450 1250 50  0000 C CNN
+F 1 "100k" H 3450 1350 60  0000 C CNN
 F 2 "Resistor_SMD:R_0402_1005Metric" H 3350 990 60  0001 L CNN
 F 3 "" H 3350 900 60  0001 L CNN
@@
 U 1 1 5F14D1BC
 P 3450 1700
-F 0 "R12" H 3550 1801 50  0000 C CNN
+F 0 "R12" H 3550 1550 50  0000 C CNN
 F 1 "280k" H 3550 1702 60  0000 C CNN
 F 2 "Resistor_SMD:R_0402_1005Metric" H 3450 1290 60  0001 L CNN
@@
 U 1 1 5F14EF13
 P 3900 1900
-F 0 "R14" H 4000 2001 50  0000 C CNN
-F 1 "200k" H 4000 1902 60  0000 C CNN
+F 0 "R14" H 4000 1750 50  0000 C CNN
+F 1 "200k" H 4000 1850 60  0000 C CNN
 F 2 "Resistor_SMD:R_0402_1005Metric" H 3900 1490 60  0001 L CNN
 F 3 "" H 3900 1400 60  0001 L CNN
@@
 U 1 1 5F14F966
 P 3450 2300
-F 0 "R13" H 3550 2401 50  0000 C CNN
-F 1 "750k" H 3550 2302 60  0000 C CNN
+F 0 "R13" H 3550 2150 50  0000 C CNN
+F 1 "750k" H 3550 2250 60  0000 C CNN
 F 2 "Resistor_SMD:R_0402_1005Metric" H 3450 1890 60  0001 L CNN
 F 3 "" H 3450 1800 60  0001 L CNN
@@
 U 1 1 5F150372
 P 3900 2500
-F 0 "R15" H 4000 2601 50  0000 C CNN
-F 1 "187k" H 4000 2502 60  0000 C CNN
+F 0 "R15" H 4000 2350 50  0000 C CNN
+F 1 "187k" H 4000 2450 60  0000 C CNN
 F 2 "Resistor_SMD:R_0402_1005Metric" H 3900 2090 60  0001 L CNN
 F 3 "" H 3900 2000 60  0001 L CNN
@@
 U 1 1 5F150C2B
 P 4400 3100
-F 0 "R18" H 4500 3201 50  0000 C CNN
-F 1 "178k" H 4500 3102 60  0000 C CNN
+F 0 "R18" H 4500 2950 50  0000 C CNN
+F 1 "178k" H 4500 3050 60  0000 C CNN
 F 2 "Resistor_SMD:R_0402_1005Metric" H 4400 2690 60  0001 L CNN
 F 3 "" H 4400 2600 60  0001 L CNN
@@
 U 1 1 5F1518D5
 P 3900 2900
-F 0 "R16" H 4000 3001 50  0000 C CNN
-F 1 "464k" H 4000 2902 60  0000 C CNN
+F 0 "R16" H 4000 2750 50  0000 C CNN
+F 1 "464k" H 4000 2850 60  0000 C CNN
 F 2 "Resistor_SMD:R_0402_1005Metric" H 3900 2490 60  0001 L CNN
 F 3 "" H 3900 2400 60  0001 L CNN
@@
 U 1 1 5F152E65
 P 3900 3500
-F 0 "R17" H 4000 3601 50  0000 C CNN
+F 0 "R17" H 4000 3300 50  0000 C CNN
 F 1 "560k" H 4000 3502 60  0000 C CNN
 F 2 "Resistor_SMD:R_0402_1005Metric" H 3900 3090 60  0001 L CNN
@@
 U 1 1 5F15318B
 P 4400 3700
-F 0 "R19" H 4500 3801 50  0000 C CNN
-F 1 "100k" H 4500 3702 60  0000 C CNN
+F 0 "R19" H 4350 3650 50  0000 C CNN
+F 1 "100k" H 4650 3650 60  0000 C CNN
 F 2 "Resistor_SMD:R_0402_1005Metric" H 4400 3290 60  0001 L CNN
 F 3 "" H 4400 3200 60  0001 L CNN
@@
 U 1 1 5F153564
 P 4400 1800
-F 0 "C9" V 4397 1810 50  0000 L CNN
-F 1 "10u" V 4496 1810 60  0000 L CNN
+F 0 "C9" V 4350 1700 50  0000 L CNN
+F 1 "10u" V 4500 1700 60  0000 L CNN
 F 2 "Capacitor_SMD:C_0603_1608Metric" H 4400 1330 60  0001 L CNN
 F 3 "" H 4400 1240 60  0001 L CNN
@@
 U 1 1 5F154046
 P 4400 2400
-F 0 "C10" V 4397 2410 50  0000 L CNN
-F 1 "10u" V 4496 2410 60  0000 L CNN
+F 0 "C10" V 4400 2300 50  0000 L CNN
+F 1 "10u" V 4500 2300 60  0000 L CNN
 F 2 "Capacitor_SMD:C_0603_1608Metric" H 4400 1930 60  0001 L CNN
 F 3 "" H 4400 1840 60  0001 L CNN
@@
 U 1 1 5F1543AE
 P 4950 3650
-F 0 "C15" V 4947 3660 50  0000 L CNN
-F 1 "10u" V 5046 3660 60  0000 L CNN
+F 0 "C15" V 4950 3550 50  0000 L CNN
+F 1 "10u" V 5050 3550 60  0000 L CNN
 F 2 "Capacitor_SMD:C_0603_1608Metric" H 4950 3180 60  0001 L CNN
 F 3 "" H 4950 3090 60  0001 L CNN
@@
 U 1 1 5F154E6A
 P 4950 2950
-F 0 "C14" V 4947 2960 50  0000 L CNN
-F 1 "10u" V 5046 2960 60  0000 L CNN
+F 0 "C14" V 4950 2850 50  0000 L CNN
+F 1 "10u" V 5050 2850 60  0000 L CNN
 F 2 "Capacitor_SMD:C_0603_1608Metric" H 4950 2480 60  0001 L CNN
 F 3 "" H 4950 2390 60  0001 L CNN
@@
 U 1 1 5F15523C
 P 4450 3800
-F 0 "C13" H 4500 3961 50  0000 C CNN
-F 1 "33p" H 4500 3862 60  0000 C CNN
+F 0 "C13" H 4600 3650 50  0000 C CNN
+F 1 "33p" H 4400 3650 60  0000 C CNN
 F 2 "Capacitor_SMD:C_0402_1005Metric" H 4450 3330 60  0001 L CNN
 F 3 "" H 4450 3240 60  0001 L CNN
@@
 U 1 1 5F155612
 P 4400 2900
-F 0 "C11" H 4450 3061 50  0000 C CNN
-F 1 "8.2p" H 4450 2962 60  0000 C CNN
+F 0 "C11" H 4550 2750 50  0000 C CNN
+F 1 "8.2p" H 4600 2850 60  0000 C CNN
 F 2 "Capacitor_SMD:C_0402_1005Metric" H 4400 2430 60  0001 L CNN
 F 3 "" H 4400 2340 60  0001 L CNN
@@
 U 1 1 5F1559FE
 P 4400 3500
-F 0 "C12" H 4450 3661 50  0000 C CNN
-F 1 "6.8p" H 4450 3562 60  0000 C CNN
+F 0 "C12" H 4550 3350 50  0000 C CNN
+F 1 "6.8p" H 4600 3450 60  0000 C CNN
 F 2 "Capacitor_SMD:C_0402_1005Metric" H 4400 3030 60  0001 L CNN
 F 3 "" H 4400 2940 60  0001 L CNN
@@
 U 1 1 5F16FAB8
 P 3350 3000
-F 0 "L1" H 3500 3249 50  0000 C CNN
+F 0 "L1" H 3500 2950 50  0000 C CNN
 F 1 "2.2uH" H 3500 3150 60  0000 C CNN
 F 2 "dsi_shield:IND_PANASONIC_ELLVEG" H 3350 3000 60  0001 C CNN
@@
 U 1 1 5F1710A3
 P 3350 3600
-F 0 "L2" H 3500 3849 50  0000 C CNN
+F 0 "L2" H 3500 3550 50  0000 C CNN
 F 1 "2.2uH" H 3500 3750 60  0000 C CNN
 F 2 "dsi_shield:IND_PANASONIC_ELLVEG" H 3350 3600 60  0001 C CNN
@@
 	4300 3600 4200 3600
 Connection ~ 4200 3600
+$Comp
+L Connector:USB_C_Plug P1
+U 1 1 5F1AC998
+P 2350 5750
+F 0 "P1" H 2457 7017 50  0000 C CNN
+F 1 "USB_C_Plug" H 2457 6926 50  0000 C CNN
+F 2 "Connector_USB:USB_C_Receptacle_Amphenol_12401548E4-2A" H 2500 5750 50  0001 C CNN
+F 3 "https://www.usb.org/sites/default/files/documents/usb_type-c.zip" H 2500 5750 50  0001 C CNN
+	1    2350 5750
+	1    0    0    -1
+$EndComp
+$Comp
+L mybays:CH340E U4
+U 1 1 5F1327DB
+P 4550 5250
+F 0 "U4" H 4550 5715 50  0000 C CNN
+F 1 "CH340E" H 4550 5624 50  0000 C CNN
+F 2 "Package_SO:MSOP-10-1EP_3x3mm_P0.5mm_EP1.68x1.88mm_ThermalVias" H 4550 4800 50  0001 C CNN
+F 3 "http://www.wch.cn/download/CH340DS1_PDF.html" H 4550 4700 50  0001 C CNN
+	1    4550 5250
+	1    0    0    -1
+$EndComp
+Wire Wire Line
+	2950 5250 4100 5250
+Wire Wire Line
+	4100 5350 3200 5350
+Wire Wire Line
+	3200 5350 3200 5450
+Wire Wire Line
+	3200 5450 2950 5450
+$Comp
+L power:GND #PWR0131
+U 1 1 5F145178
+P 4100 5600
+F 0 "#PWR0131" H 4100 5350 50  0001 C CNN
+F 1 "GND" H 4105 5427 50  0000 C CNN
+F 2 "" H 4100 5600 50  0001 C CNN
+F 3 "" H 4100 5600 50  0001 C CNN
+	1    4100 5600
+	1    0    0    -1
+$EndComp
+$Comp
+L power:GND #PWR0132
+U 1 1 5F145B88
+P 2150 7550
+F 0 "#PWR0132" H 2150 7300 50  0001 C CNN
+F 1 "GND" H 2155 7377 50  0000 C CNN
+F 2 "" H 2150 7550 50  0001 C CNN
+F 3 "" H 2150 7550 50  0001 C CNN
+	1    2150 7550
+	1    0    0    -1
+$EndComp
+$Comp
+L power:+5V #PWR0133
+U 1 1 5F147659
+P 4000 4900
+F 0 "#PWR0133" H 4000 4750 50  0001 C CNN
+F 1 "+5V" H 4015 5073 50  0000 C CNN
+F 2 "" H 4000 4900 50  0001 C CNN
+F 3 "" H 4000 4900 50  0001 C CNN
+	1    4000 4900
+	1    0    0    -1
+$EndComp
+Wire Wire Line
+	4100 5050 4000 5050
+Wire Wire Line
+	4000 5050 4000 4900
+$Comp
+L power:+5V #PWR0134
+U 1 1 5F14B9DC
+P 3000 4550
+F 0 "#PWR0134" H 3000 4400 50  0001 C CNN
+F 1 "+5V" H 3015 4723 50  0000 C CNN
+F 2 "" H 3000 4550 50  0001 C CNN
+F 3 "" H 3000 4550 50  0001 C CNN
+	1    3000 4550
+	1    0    0    -1
+$EndComp
+Wire Wire Line
+	2950 4750 3000 4750
+Wire Wire Line
+	3000 4750 3000 4650
+$Comp
+L dsi_shield:Cap C17
+U 1 1 5F150745
+P 3800 5050
+F 0 "C17" H 3800 4800 50  0000 C CNN
+F 1 "100n" H 3850 5112 60  0000 C CNN
+F 2 "Capacitor_SMD:C_0402_1005Metric" H 3800 4580 60  0001 L CNN
+F 3 "" H 3800 4490 60  0001 L CNN
+F 4 "8-Jun-2000" H 3800 4400 60  0001 L CNN "字段4"
+F 5 "17-Jul-2002" H 3800 4310 60  0001 L CNN "字段5"
+F 6 "Re-released for DXP Platform." H 3800 4220 60  0001 L CNN "字段6"
+F 7 "RAD-0.3" H 3800 4130 60  0001 L CNN "字段7"
+F 8 "Altium Limited" H 3800 4040 60  0001 L CNN "字段8"
+F 9 "Yes" H 3800 3950 60  0001 L CNN "字段9"
+F 10 "100n" H 3850 5106 50  0001 C CNN "字段10"
+F 11 "=Value" H 3800 3770 60  0001 L CNN "字段11"
+	1    3800 5050
+	1    0    0    -1
+$EndComp
+$Comp
+L power:GND #PWR0135
+U 1 1 5F151F09
+P 3600 5100
+F 0 "#PWR0135" H 3600 4850 50  0001 C CNN
+F 1 "GND" H 3605 4927 50  0000 C CNN
+F 2 "" H 3600 5100 50  0001 C CNN
+F 3 "" H 3600 5100 50  0001 C CNN
+	1    3600 5100
+	-1   0    0    1
+$EndComp
+Wire Wire Line
+	4000 5150 4100 5150
+Wire Wire Line
+	3700 5150 3600 5150
+Wire Wire Line
+	3600 5150 3600 5100
+Wire Wire Line
+	4100 5450 4100 5600
+$Comp
+L dsi_shield:Cap C16
+U 1 1 5F15EA9B
+P 3150 4550
+F 0 "C16" H 3150 4300 50  0000 C CNN
+F 1 "10u" H 3200 4612 60  0000 C CNN
+F 2 "Capacitor_SMD:C_0603_1608Metric" H 3150 4080 60  0001 L CNN
+F 3 "" H 3150 3990 60  0001 L CNN
+F 4 "8-Jun-2000" H 3150 3900 60  0001 L CNN "字段4"
+F 5 "17-Jul-2002" H 3150 3810 60  0001 L CNN "字段5"
+F 6 "Re-released for DXP Platform." H 3150 3720 60  0001 L CNN "字段6"
+F 7 "RAD-0.3" H 3150 3630 60  0001 L CNN "字段7"
+F 8 "Altium Limited" H 3150 3540 60  0001 L CNN "字段8"
+F 9 "Yes" H 3150 3450 60  0001 L CNN "字段9"
+F 10 "100n" H 3200 4606 50  0001 C CNN "字段10"
+F 11 "=Value" H 3150 3270 60  0001 L CNN "字段11"
+	1    3150 4550
+	1    0    0    -1
+$EndComp
+$Comp
+L power:GND #PWR0136
+U 1 1 5F1601F5
+P 3350 4750
+F 0 "#PWR0136" H 3350 4500 50  0001 C CNN
+F 1 "GND" H 3355 4577 50  0000 C CNN
+F 2 "" H 3350 4750 50  0001 C CNN
+F 3 "" H 3350 4750 50  0001 C CNN
+	1    3350 4750
+	1    0    0    -1
+$EndComp
+Wire Wire Line
+	3350 4750 3350 4650
+Wire Wire Line
+	3050 4650 3000 4650
+Connection ~ 3000 4650
+Wire Wire Line
+	3000 4650 3000 4550
+Text GLabel 5050 5050 2    50   Input ~ 0
+RXD
+Text GLabel 5050 5150 2    50   Input ~ 0
+TXD
+Wire Wire Line
+	5000 5050 5050 5050
+Wire Wire Line
+	5000 5150 5050 5150
 $EndSCHEMATC

Commit message: 20200808
Parts:
- added C42, C46, C47: 4.7u, Capacitor_SMD:C_0805_2012Metric, symbol dsi_shield:Cap
- added C43, C44, C48: 1u, Capacitor_SMD:C_0603_1608Metric_Pad1.05x0.95mm_HandSolder, symbol dsi_shield:Cap
- added C45, C49: 22p, Capacitor_SMD:C_0402_1005Metric, symbol dsi_shield:Cap
- added D6, D7, D8, D9: Diode_Schottky, dsi_shield:SOD3715X145N, symbol dsi_shield:Diode_Schottky
- added IC4, IC5: SOT95P275X110-5N, mybays:SOT95P275X110-5N, symbol dsi_shield:TPS61041
- added L3, L4: 4.7uH, dsi_shield:IND_PANASONIC_ELLVEG, symbol dsi_shield:DLCSM0315D-2R2-K
- added R35, R37: 0, Resistor_SMD:R_0402_1005Metric, symbol dsi_shield:Res1
- added R41, R42, R44: 100k, Resistor_SMD:R_0402_1005Metric, symbol dsi_shield:Res1
- added R43, R45: 27k, Resistor_SMD:R_0402_1005Metric, symbol dsi_shield:Res1
Connections:
- net +1V8: now also R35.1
- net +2V5: now also R37.1
- net +3V3: now also C42.1, C47.1, IC4.5 (VIN), IC5.4 (EN), IC5.5 (VIN), L3.1, L4.1
- net GND: now also P1.A1 (GND), P1.A12 (GND), P1.B1 (GND), P1.B12 (GND), P1.S1 (SHIELD), C42.2, C44.2, C46.2, C47.2, C48.2, D7.1 (C), IC4.2 (GND), IC5.2 (GND), R41.2, R43.2, R45.2
- net CPU_RST: now reaches U4.4 (~RTS~)
- net RXD renamed DBG_RX
- net TXD renamed DBG_TX
- new net: C43.2, D6.2 (A), IC4.1 (SW), L3.2
- new net: C43.1, D7.2 (A), D8.1 (C)
- new net: D9.2 (A), IC5.1 (SW), L4.2
- new net LCD_BL_A: C48.1, C49.1, D9.1 (C), R44.1
- new net LCD_BL_FB: C49.2, IC5.3 (FB), R44.2, R45.1
- new net LCD_BOOST_FB: C45.2, IC4.3 (FB), R42.2, R43.1
- new net LCD_MVDD: C46.1, D8.2 (A)
- new net LCD_PVDD: C44.1, C45.1, D6.1 (C), R42.1
- new net LCD_PWREN: IC4.4 (EN), R41.1
- new net V_DDR: R35.2, R37.2
- no-connect marks 0 -> 14
