File: dsi-shield-bga/connector.sch (KiCad schematic (older format))
At the start: 1 part, among them CN1 Header_6

Commit message: pin head
Parts:
- added J4, J5: Conn_02x36_Odd_Even, Connector_PinSocket_2.54mm:PinSocket_2x36_P2.54mm_Vertical, symbol Connector_Generic:Conn_02x36_Odd_Even
Changed lines of the file:
@@
 	0    1    1    0
 $EndComp
+$Comp
+L Connector_Generic:Conn_02x36_Odd_Even J4
+U 1 1 5F43B64D
+P 3950 3950
+F 0 "J4" H 4000 5867 50  0000 C CNN
+F 1 "Conn_02x36_Odd_Even" H 4000 5776 50  0000 C CNN
+F 2 "Connector_PinSocket_2.54mm:PinSocket_2x36_P2.54mm_Vertical" H 3950 3950 50  0001 C CNN
+F 3 "~" H 3950 3950 50  0001 C CNN
+	1    3950 3950
+	1    0    0    -1
+$EndComp
+$Comp
+L Connector_Generic:Conn_02x36_Odd_Even J5
+U 1 1 5F440AF6
+P 4900 3950
+F 0 "J5" H 4950 5867 50  0000 C CNN
+F 1 "Conn_02x36_Odd_Even" H 4950 5776 50  0000 C CNN
+F 2 "Connector_PinSocket_2.54mm:PinSocket_2x36_P2.54mm_Vertical" H 4900 3950 50  0001 C CNN
+F 3 "~" H 4900 3950 50  0001 C CNN
+	1    4900 3950
+	1    0    0    -1
+$EndComp
 $EndSCHEMATC
