File: dsi-shield-bga/dsi-shield-bga.kicad_pcb (KiCad board)
At the start: 2 copper layers, 100 x 100 mm, 148 parts, among them CN1 Header_6, IC1 LM26480, IC10 MT46V32M16P-5B:F, IC2 M25P80-VMN6P, IC3 25MHz, IC4 SOT95P275X110-5N, IC5 SOT95P275X110-5N, J1 10118241-001RLF, J2 Conn_02x15_Odd_Even, P1 USB_C_Plug, Q1 2N7002, Q2 2N7002, Q3 Q_BSS84, Q4 2N7002, U1 XC6SLX16-FTG256, U2 K4X1G163PE, U4 CH340E

Commit message: pin head
Parts:
- removed IC10: MT46V32M16P-5B:F, dsi_shield:TSOP66
- added IC6: MT46V64M16P-5B_F, dsi_shield:TSOP66, B.Cu at (85.0, 84.0)
- added J3: Conn_02x05_Odd_Even, mybays_connector:debugger_2x05_P1.27mm_Vertical, F.Cu at (201.0, 114.0)
- added J4: Conn_02x36_Odd_Even, Connector_PinSocket_2.54mm:PinSocket_2x35_P2.54mm_Vertical, F.Cu at (55.0, 56.0)
- added J5: Conn_02x36_Odd_Even, Connector_PinSocket_2.54mm:PinSocket_2x35_P2.54mm_Vertical, F.Cu at (56.0, 110.0)
- moved U1 1.50 mm to (113.5, 84.5)
Connections:
- U1 pad E15: Net-(U1-PadE15) -> DSI_HS_0_P
- U1 pad E16: Net-(U1-PadE16) -> DSI_HS_0_N
- U1 pad F15: Net-(U1-PadF15) -> DSI_LP_0_P
- U1 pad F16: Net-(U1-PadF16) -> DSI_LP_0_N
- U1 pad G14: Net-(U1-PadG14) -> DSI_HS_1_P
- U1 pad G16: Net-(U1-PadG16) -> DSI_HS_1_N
- U1 pad H15: DSI_HS_CLK_P -> Net-(U1-PadH15)
- U1 pad H16: DSI_HS_CLK_N -> Net-(U1-PadH16)
- U1 pad J14: DSI_LP_CLK_P -> DSI_LP_1_P
- U1 pad J16: DSI_LP_CLK_N -> DSI_LP_1_N
- U1 pad K15: Net-(U1-PadK15) -> DSI_HS_CLK_P
- U1 pad K16: Net-(U1-PadK16) -> DSI_HS_CLK_N
- U1 pad L14: Net-(U1-PadL14) -> DSI_LP_CLK_P
- U1 pad L16: Net-(U1-PadL16) -> DSI_LP_CLK_N
- U1 pad M15: Net-(U1-PadM15) -> DSI_HS_2_P
- U1 pad M16: Net-(U1-PadM16) -> DSI_HS_2_N
- U1 pad N14: Net-(U1-PadN14) -> DSI_LP_2_P
- U1 pad N16: Net-(U1-PadN16) -> DSI_LP_2_N
- U1 pad P15: Net-(U1-PadP15) -> DSI_HS_3_P
- U1 pad P16: Net-(U1-PadP16) -> DSI_HS_3_N
- U1 pad R15: Net-(U1-PadR15) -> DSI_LP_3_P
- U1 pad R16: Net-(U1-PadR16) -> DSI_LP_3_N
Routing:
- net GND: track 48.8 -> 0.00 mm, vias 69 -> 0
- net +3V3: track 36.1 -> 0.00 mm, vias 51 -> 0
- net +1V2: track 17.0 -> 0.00 mm, vias 24 -> 0
- net +1V8: track 12.7 -> 0.00 mm, vias 18 -> 0
- net V_DDR: track 10.6 -> 0.00 mm, vias 15 -> 0
- net Net-(R36-Pad1): track 2.12 -> 0.00 mm, vias 3 -> 0
- net Net-(R27-Pad1): track 2.12 -> 0.00 mm, vias 3 -> 0
- net Net-(D5-Pad2): track 2.12 -> 0.00 mm, vias 3 -> 0
- net FPGA_TDO: track 2.12 -> 0.00 mm, vias 3 -> 0
- net FPGA_TDI: track 2.12 -> 0.00 mm, vias 3 -> 0
- net FPGA_TCK: track 2.12 -> 0.00 mm, vias 3 -> 0
- net DSI_RESET_N: track 2.12 -> 0.00 mm, vias 3 -> 0
- net DSI_LP_CLK_P: track 2.12 -> 0.00 mm, vias 3 -> 0
- net DSI_HS_CLK_P: track 2.12 -> 0.00 mm, vias 3 -> 0
- net DSI_GPIO1: track 2.12 -> 0.00 mm, vias 3 -> 0
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